Commit message: model.sdf/urdf fixes and launch file fixes

File: isabelle_sim/models/isabelle/model.urdf (robot description, URDF)
Before this commit: robot isabelle, 7 links, 6 joints
Joints:
- joint back_left_wheel_hinge: origin xyz=0.1 0.13 0.1 rpy=0 0 0 -> xyz=0.12 0.0762 0.2 rpy=0 0 0
- joint back_right_wheel_hinge: origin xyz=0.1 -0.13 0.1 rpy=0 0 0 -> xyz=0.12 -0.0762 0.2 rpy=0 0 0
- joint front_left_wheel_hinge: origin xyz=-0.1 0.13 0.1 rpy=0 0 0 -> xyz=-0.12 0.0762 0.2 rpy=0 0 0
- joint front_right_wheel_hinge: origin xyz=-0.1 -0.13 0.1 rpy=0 0 0 -> xyz=-0.12 -0.0762 0.2 rpy=0 0 0
- joint imu joint: origin xyz=0 0 0.01 -> xyz=0 0 0.1

Commit message: fixed robot dimensions

File: isabelle_sim/models/isabelle/model.urdf (robot description, URDF)
Before this commit: robot isabelle, 7 links, 6 joints
Links:
- link camera_link: geometry collision box size=0.02 0.09 0.02; visual box size=0.02 0.09 0.02
- link chassis: geometry collision box size=.254 .1524 .04; visual box size=.254 .1524 .04
Joints:
- joint back_left_wheel_hinge: origin xyz=0.12 0.0762 0.2 rpy=0 0 0 -> xyz=-.09779 -.09 -.01079 rpy=0 0 0
- joint back_right_wheel_hinge: origin xyz=0.12 -0.0762 0.2 rpy=0 0 0 -> xyz=-.09779 .09 -.01079 rpy=0 0 0
- joint front_left_wheel_hinge: origin xyz=-0.12 0.0762 0.2 rpy=0 0 0 -> xyz=.09779 -0.09 -.01079 rpy=0 0 0
- joint front_right_wheel_hinge: origin xyz=-0.12 -0.0762 0.2 rpy=0 0 0 -> xyz=.09779 0.09 -.01079 rpy=0 0 0

Commit message: Adds skid steer drive controller

File: isabelle_sim/models/isabelle/model.urdf (robot description, URDF)
Before this commit: robot isabelle, 7 links, 6 joints
Links:
- link chassis: mass 2.25 -> None
Joints:
- joint back_left_wheel_hinge: origin xyz=-.09779 -.09 -.01079 rpy=0 0 0 -> xyz=-.09779 -.0762 -.01079 rpy=0 0 0
- joint back_right_wheel_hinge: origin xyz=-.09779 .09 -.01079 rpy=0 0 0 -> xyz=-.09779 .0762 -.01079 rpy=0 0 0
- joint front_left_wheel_hinge: origin xyz=.09779 -0.09 -.01079 rpy=0 0 0 -> xyz=.09779 -.0762 -.01079 rpy=0 0 0
- joint front_right_wheel_hinge: origin xyz=.09779 0.09 -.01079 rpy=0 0 0 -> xyz=.09779 .0762 -.01079 rpy=0 0 0

Commit message: Fixes some tf issues

File: isabelle_sim/models/isabelle/model.urdf (robot description, URDF)
Before this commit: robot isabelle, 7 links, 6 joints
Links:
- link back_left_wheel: geometry collision cylinder length=.0254 radius=.02921; visual cylinder length=.0254 radius=.02921
- link back_right_wheel: geometry collision cylinder length=.0254 radius=.02921; visual cylinder length=.0254 radius=.02921
- link front_left_wheel: geometry collision cylinder length=.0254 radius=.02921; visual cylinder length=.0254 radius=.02921
- link front_right_wheel: geometry collision cylinder length=.0254 radius=.02921; visual cylinder length=.0254 radius=.02921

Commit message: Fixes model in gazebo

File: isabelle_sim/models/isabelle/model.urdf (robot description, URDF)
Before this commit: robot isabelle, 7 links, 6 joints
Joints:
- joint back_left_wheel_hinge: origin xyz=-.09779 -.0762 -.01079 rpy=0 0 0 -> xyz=-.09779 -.09 -.01079 rpy=0 0 0
- joint back_right_wheel_hinge: origin xyz=-.09779 .0762 -.01079 rpy=0 0 0 -> xyz=-.09779 .09 -.01079 rpy=0 0 0
- joint camera_joint: origin xyz=0.0 0.0 0.385 rpy=1.5708 3.14159 1.5708 -> xyz=0.0 0.0 0.03 rpy=1.5708 1.5708 1.5708
- joint front_left_wheel_hinge: origin xyz=.09779 -.0762 -.01079 rpy=0 0 0 -> xyz=.09779 -.09 -.01079 rpy=0 0 0
- joint front_right_wheel_hinge: origin xyz=.09779 .0762 -.01079 rpy=0 0 0 -> xyz=.09779 .09 -.01079 rpy=0 0 0
- joint imu joint: origin xyz=0 0 0.1 -> xyz=0 0 0.045

Commit message: Adds motors.py from UGV sim, and fixes inertia issues.

File: isabelle_sim/models/isabelle/model.urdf (robot description, URDF)
Before this commit: robot isabelle, 7 links, 6 joints
Links:
- link chassis: mass None -> 0.68
Joints:
- joint camera_joint: origin xyz=0.0 0.0 0.03 rpy=1.5708 1.5708 1.5708 -> xyz=0.2 0.0 0.03 rpy=1.5708 1.5708 1.5708

Commit message: Adds lidar and fixes some skid steering issues.

File: isabelle_sim/models/isabelle/model.urdf (robot description, URDF)
Before this commit: robot isabelle, 7 links, 6 joints
Links:
- added link hokuyo_link; collision box size=0.0508 0.0508 0.0762; visual box size=0.0508 0.0508 0.0762
Joints:
- added joint hokuyo_joint: type fixed, parent chassis, child hokuyo_link, origin xyz=0.0 0.0 0.0481 rpy=0 0 0, axis 0 1 0, limit lower=0.0 upper=0.0 effort=0.0 velocity=0.0
- joint camera_joint: origin xyz=0.2 0.0 0.03 rpy=1.5708 1.5708 1.5708 -> xyz=-0.1 0.0 0.03 rpy=1.5708 1.5708 1.5708
- joint imu joint: origin xyz=0 0 0.045 -> xyz=-0.1 0 0.045

Commit message: Added config files for ekf_localization and slam toolbox node

File: isabelle_sim/models/isabelle/model.urdf (robot description, URDF)
Before this commit: robot isabelle, 8 links, 7 joints
Joints:
- joint hokuyo_joint: origin xyz=0.0 0.0 0.0481 rpy=0 0 0 -> xyz=0.0 0.0 0.0481 rpy=0 0 1.5708

Commit message: Uses Hector_mapping, adds move_base goal setter, configures nav_stack, finishes xacro migration. TLDR: Does the thing.

File: isabelle_sim/models/isabelle/model.urdf (robot description, URDF)
Before this commit: robot isabelle, 8 links, 7 joints
Links:
- removed link back_left_wheel
- removed link back_right_wheel
- removed link camera_link
- removed link chassis
- added link back_left_caster, mass .045; collision sphere radius=.02921; visual sphere radius=.02921
- added link back_right_caster, mass .045; collision sphere radius=.02921; visual sphere radius=.02921
- added link base_link, mass 0.68; collision box size=.254 .1524 .04; visual box size=.254 .1524 .04
Joints:
- removed joint back_left_wheel_hinge
- removed joint back_right_wheel_hinge
- removed joint camera_joint
- added joint back_left_caster_hinge: type revolute, parent base_link, child back_left_caster, origin xyz=.09779 -.09 -.01079 rpy=0 0 0, axis 0 1 0, limit lower=0 upper=0 effort=0 velocity=0
- added joint back_right_caster_hinge: type revolute, parent base_link, child back_right_caster, origin xyz=.09779 .09 -.01079 rpy=0 0 0, axis 0 1 0, limit lower=0 upper=0 effort=0 velocity=0
- joint front_left_wheel_hinge: origin xyz=.09779 -.09 -.01079 rpy=0 0 0 -> xyz=-.09779 -.09 -.01079 rpy=0 0 0; parent chassis -> base_link
- joint front_right_wheel_hinge: origin xyz=.09779 .09 -.01079 rpy=0 0 0 -> xyz=-.09779 .09 -.01079 rpy=0 0 0; parent chassis -> base_link
- joint hokuyo_joint: origin xyz=0.0 0.0 0.0481 rpy=0 0 1.5708 -> xyz=0.0 0.0 0.0481 rpy=0 0 0; parent chassis -> base_link
- joint imu joint: origin xyz=-0.1 0 0.045 -> xyz=0 0 0; parent chassis -> base_link
